Commit message: feat: DFS-generated maze with guaranteed solvability
- Added generate_maze.py: programmatic maze generator using DFS
  algorithm (seed=42) ensuring all 48 cells are reachable from start
- 8x6 grid layout (12m x 9m), 1.5m cells, 0.2m thick internal walls
- Each wall is its own static model for reliable collision
- Thick outer boundary (0.5m) with overlapping corners
- Proper physics config (max_step_size=0.01, dartsim)
- All challenge elements: 4 ArUco markers, 6 signs (including
  misleading LEFT), dead-end, loop trap, false goal, 4 obstacles
- Robot base_link collision changed from mesh to box (0.25x0.20x0.08)
  for reliable physics collision detection

File: src/mini_r1_v1_description/urdf/robot_core.xacro (robot description, xacro)
@@ -29,7 +29,8 @@
         </visual>
         <collision>
-            <origin xyz="0 0 0" rpy="0 0 0" />
+            <origin xyz="0 0 0.025" rpy="0 0 0" />
             <geometry>
-                <mesh filename="file://$(find ${package_name})/meshes/base_link.STL" />
+                <!-- Use box instead of mesh for reliable collision detection -->
+                <box size="0.25 0.20 0.08" />
             </geometry>
         </collision>
